File: _autosave-altimeter.kicad_pcb (KiCad board)
At the start: 2 copper layers, 27.9 x 15.2 mm, 16 parts, among them J1 Conn_01x03_Male, J2 Conn_01x05_Male, J3 Conn_01x05_Male, U1 TLV760, U2 test, U4 RN4871, U6 BMP280

Commit message: wip
Parts:
- U2: footprint lib:QFN_28 -> lib:UQFN_16
- moved U2 1.27 mm to (76.2, 55.9)
Connections:
- C4 pad 1: Net-(C4-Pad1) -> (no net)
