File: _saved_altimeter.sch (KiCad schematic (older format))
At the start: 16 parts, among them J1 Conn_01x03_Male, J2 Conn_01x05_Male, J3 Conn_01x05_Male, U1 TLV760, U2 test, U4 RN4871, U6 BMP280

Commit message: wip
Parts:
- C1, C2, C3, C4, C5, C7: footprint Capacitors_SMD:C_0805_HandSoldering -> Capacitors_SMD:C_0603
- J2, J3: footprint Pin_Headers:Pin_Header_Straight_1x05_Pitch2.54mm -> lib:pin5
- R1, R2, R3: footprint Resistors_SMD:R_0805_HandSoldering -> Resistors_SMD:R_0603
- U2: footprint lib:QFN_28 -> lib:UQFN_16
Changed lines of the file:
@@
 F 0 "U2" H 3250 2400 60  0000 C CNN
 F 1 "test" H 3250 2400 60  0000 C CNN
-F 2 "lib:QFN_28" H 3250 2400 60  0001 C CNN
+F 2 "lib:UQFN_16" H 3250 2400 60  0001 C CNN
 F 3 "" H 3250 2400 60  0001 C CNN
 	1    3250 2400
@@
 F 0 "C2" H 2075 2750 50  0000 L CNN
 F 1 "0.1u" H 2075 2550 50  0000 L CNN
-F 2 "Capacitors_SMD:C_0805_HandSoldering" H 2088 2500 50  0001 C CNN
+F 2 "Capacitors_SMD:C_0603" H 2088 2500 50  0001 C CNN
 F 3 "" H 2050 2650 50  0001 C CNN
 	1    2050 2650
@@
 F 0 "C5" H 4175 1800 50  0000 L CNN
 F 1 "0.1u" H 4175 1600 50  0000 L CNN
-F 2 "Capacitors_SMD:C_0805_HandSoldering" H 4188 1550 50  0001 C CNN
+F 2 "Capacitors_SMD:C_0603" H 4188 1550 50  0001 C CNN
 F 3 "" H 4150 1700 50  0001 C CNN
 	1    4150 1700
@@
 F 0 "R3" V 2380 1700 50  0000 C CNN
 F 1 "10k" V 2300 1700 50  0000 C CNN
-F 2 "Resistors_SMD:R_0805_HandSoldering" V 2230 1700 50  0001 C CNN
+F 2 "Resistors_SMD:R_0603" V 2230 1700 50  0001 C CNN
 F 3 "" H 2300 1700 50  0001 C CNN
 	1    2300 1700
@@
 F 0 "C4" H 4075 2600 50  0000 L CNN
 F 1 "10u" H 4075 2400 50  0000 L CNN
-F 2 "Capacitors_SMD:C_0805_HandSoldering" H 4088 2350 50  0001 C CNN
+F 2 "Capacitors_SMD:C_0603" H 4088 2350 50  0001 C CNN
 F 3 "" H 4050 2500 50  0001 C CNN
 	1    4050 2500
@@
 U1RX
 $Comp
-L +3.3V #PWR011
+L +3.3V #PWR07
 U 1 1 5ABFEDB5
 P 5550 5200
-F 0 "#PWR011" H 5550 5050 50  0001 C CNN
+F 0 "#PWR07" H 5550 5050 50  0001 C CNN
 F 1 "+3.3V" H 5550 5340 50  0000 C CNN
 F 2 "" H 5550 5200 50  0001 C CNN
@@
 $EndComp
 $Comp
-L VSS #PWR012
+L VSS #PWR08
 U 1 1 5ABFEDDD
 P 5650 5350
-F 0 "#PWR012" H 5650 5200 50  0001 C CNN
+F 0 "#PWR08" H 5650 5200 50  0001 C CNN
 F 1 "VSS" H 5650 5500 50  0000 C CNN
 F 2 "" H 5650 5350 50  0001 C CNN
@@
 	5250 5350 5650 5350
 $Comp
-L VSS #PWR013
+L VSS #PWR09
 U 1 1 5ABFF34C
 P 4150 5100
-F 0 "#PWR013" H 4150 4950 50  0001 C CNN
+F 0 "#PWR09" H 4150 4950 50  0001 C CNN
 F 1 "VSS" H 4150 5250 50  0000 C CNN
 F 2 "" H 4150 5100 50  0001 C CNN
@@
 F 0 "J2" H 1150 4300 50  0000 C CNN
 F 1 "Conn_01x05_Male" H 1150 3700 50  0000 C CNN
-F 2 "Pin_Headers:Pin_Header_Straight_1x05_Pitch2.54mm" H 1150 4000 50  0001 C CNN
+F 2 "lib:pin5" H 1150 4000 50  0001 C CNN
 F 3 "" H 1150 4000 50  0001 C CNN
 	1    1150 4000
@@
 	2450 2300 2650 2300
 $Comp
-L +3.3V #PWR014
+L +3.3V #PWR010
 U 1 1 5AC12FB0
 P 2200 3900
-F 0 "#PWR014" H 2200 3750 50  0001 C CNN
+F 0 "#PWR010" H 2200 3750 50  0001 C CNN
 F 1 "+3.3V" H 2200 4040 50  0000 C CNN
 F 2 "" H 2200 3900 50  0001 C CNN
@@
 $EndComp
 $Comp
-L VSS #PWR015
+L VSS #PWR011
 U 1 1 5AC12FCE
 P 2450 4000
-F 0 "#PWR015" H 2450 3850 50  0001 C CNN
+F 0 "#PWR011" H 2450 3850 50  0001 C CNN
 F 1 "VSS" H 2450 4150 50  0000 C CNN
 F 2 "" H 2450 4000 50  0001 C CNN
@@
 	3850 1900 6050 1900
 $Comp
-L +3.3V #PWR016
+L +3.3V #PWR012
 U 1 1 5AC190CB
 P 8150 900
-F 0 "#PWR016" H 8150 750 50  0001 C CNN
+F 0 "#PWR012" H 8150 750 50  0001 C CNN
 F 1 "+3.3V" H 8150 1040 50  0000 C CNN
 F 2 "" H 8150 900 50  0001 C CNN
@@
 $EndComp
 $Comp
-L VSS #PWR017
+L VSS #PWR013
 U 1 1 5AC190DC
 P 8400 2150
-F 0 "#PWR017" H 8400 2000 50  0001 C CNN
+F 0 "#PWR013" H 8400 2000 50  0001 C CNN
 F 1 "VSS" H 8400 2300 50  0000 C CNN
 F 2 "" H 8400 2150 50  0001 C CNN
@@
 $EndComp
 $Comp
-L +3.3V #PWR018
+L +3.3V #PWR014
 U 1 1 5AC19B3B
 P 3150 5400
-F 0 "#PWR018" H 3150 5250 50  0001 C CNN
+F 0 "#PWR014" H 3150 5250 50  0001 C CNN
 F 1 "+3.3V" H 3150 5540 50  0000 C CNN
 F 2 "" H 3150 5400 50  0001 C CNN
@@
 	3150 5400 3150 5750
 $Comp
-L VSS #PWR019
+L VSS #PWR015
 U 1 1 5AC19BAA
 P 2550 6050
-F 0 "#PWR019" H 2550 5900 50  0001 C CNN
+F 0 "#PWR015" H 2550 5900 50  0001 C CNN
 F 1 "VSS" H 2550 6200 50  0000 C CNN
 F 2 "" H 2550 6050 50  0001 C CNN
@@
 F 0 "R2" V 2180 6050 50  0000 C CNN
 F 1 "100k" V 2100 6050 50  0000 C CNN
-F 2 "Resistors_SMD:R_0805_HandSoldering" V 2030 6050 50  0001 C CNN
+F 2 "Resistors_SMD:R_0603" V 2030 6050 50  0001 C CNN
 F 3 "" H 2100 6050 50  0001 C CNN
 	1    2100 6050
@@
 F 0 "R1" V 1830 6050 50  0000 C CNN
 F 1 "200k" V 1750 6050 50  0000 C CNN
-F 2 "Resistors_SMD:R_0805_HandSoldering" V 1680 6050 50  0001 C CNN
+F 2 "Resistors_SMD:R_0603" V 1680 6050 50  0001 C CNN
 F 3 "" H 1750 6050 50  0001 C CNN
 	1    1750 6050
@@
 F 0 "J3" H 5800 6250 50  0000 C CNN
 F 1 "Conn_01x05_Male" H 6050 5650 50  0000 C CNN
-F 2 "Pin_Headers:Pin_Header_Straight_1x05_Pitch2.54mm" H 5800 5950 50  0001 C CNN
+F 2 "lib:pin5" H 5800 5950 50  0001 C CNN
 F 3 "" H 5800 5950 50  0001 C CNN
 	1    5800 5950
@@
 F 0 "C1" H 1525 6200 50  0000 L CNN
 F 1 "10u" H 1525 6000 50  0000 L CNN
-F 2 "Capacitors_SMD:C_0805_HandSoldering" H 1538 5950 50  0001 C CNN
+F 2 "Capacitors_SMD:C_0603" H 1538 5950 50  0001 C CNN
 F 3 "" H 1500 6100 50  0001 C CNN
 	1    1500 6100
@@
 F 0 "C3" H 3175 6000 50  0000 L CNN
 F 1 "10u" H 3175 5800 50  0000 L CNN
-F 2 "Capacitors_SMD:C_0805_HandSoldering" H 3188 5750 50  0001 C CNN
+F 2 "Capacitors_SMD:C_0603" H 3188 5750 50  0001 C CNN
 F 3 "" H 3150 5900 50  0001 C CNN
 	1    3150 5900
@@
 F 0 "C7" H 9325 1500 50  0000 L CNN
 F 1 ".1u" H 9325 1300 50  0000 L CNN
-F 2 "Capacitors_SMD:C_0805_HandSoldering" H 9338 1250 50  0001 C CNN
+F 2 "Capacitors_SMD:C_0603" H 9338 1250 50  0001 C CNN
 F 3 "" H 9300 1400 50  0001 C CNN
 	1    9300 1400

Commit message: wip
Parts:
- removed C2: 0.1u, Capacitors_SMD:C_0603, symbol CP
- removed C4: 10u, Capacitors_SMD:C_0603, symbol CP
- removed U2: test, lib:UQFN_16, symbol dsPIC33_qfn
- added B1: 1632-holder, lib:1632-holder, symbol 1632-holder
- added U2: PIC16F15325, lib:UQFN_16, symbol PIC16F15325
Connections:
- net labels removed: Pyro1, Pyro2
- wire segments 82 -> 73
Other:
- moved on the sheet: C5, R3
