File: altimeter.sch (KiCad schematic (older format))
At the start: 23 parts, among them J1 Conn_01x03_Male, J2 Conn_01x05_Male, J3 Conn_01x05_Male, J4 Conn_01x03_Male, Q1 Q_NMOS_DGS, U1 TLV760, U2 test, U3 accel, U4 RN4871, U5 EEPROM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

Commit message: Dev3
Parts:
- removed C6: 1u, Capacitors_SMD:C_0805_HandSoldering, symbol CP
- removed U3: accel, SMD_Packages:SOIC-8-N, symbol accel
- added J5, J6: Conn_01x01_Male, lib:2-56_hole, symbol Conn_01x01_Male
- added Q2: Q_NMOS_DGS, TO_SOT_Packages_SMD:SOT-23, symbol DMN2046U
- added R6: 100k, Resistors_SMD:R_0603, symbol R
- C1, C2, C3, C4, C5, C7: footprint Capacitors_SMD:C_0805_HandSoldering -> Capacitors_SMD:C_0603
- J1: footprint Pin_Headers:Pin_Header_Straight_1x03_Pitch2.54mm -> Pin_Headers:Pin_Header_Straight_1x02_Pitch2.54mm; symbol Conn_01x03_Male -> Conn_01x02_Male
- J4: footprint Pin_Headers:Pin_Header_Straight_1x03_Pitch2.54mm -> Pin_Headers:Pin_Header_Straight_1x04_Pitch2.54mm; symbol Conn_01x03_Male -> Conn_01x04_Male
- Q1: symbol Q_NMOS_DGS -> DMN2046U
- R1, R2, R3, R4, R5: footprint Resistors_SMD:R_0805_HandSoldering -> Resistors_SMD:R_0603
Connections:
- net DEBUG: now also J5.1 (Pin_1); no longer J1.1 (Pin_1)
- net Pyro1: now also Q1.1 (G); no longer Q1.2 (G)
- net Pyro2: now also Q2.1 (G), R6.2
- net VIN: now also J1.1 (Pin_1); no longer J1.2 (Pin_2)
- net VSS: now also J1.2 (Pin_2), Q1.2 (S), J6.1 (Pin_1), Q2.2 (S), R6.1; no longer J1.3 (Pin_3), Q1.3 (S)
- net at J4.2 (Pin_2): now also J4.1 (Pin_1), R5.1; no longer Q1.1 (D)
- net at J4.3 (Pin_3): now also Q1.3 (D)
- new net: J4.4 (Pin_4), Q2.3 (D)
