File: altimeter.sch (KiCad schematic (older format))
At the start: 23 parts, among them J1 Conn_01x03_Male, J2 Conn_01x05_Male, J3 Conn_01x05_Male, J4 Conn_01x03_Male, Q1 Q_NMOS_DGS, U1 TLV760, U2 test, U3 accel, U4 RN4871, U5 EEPROM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

Commit message: wip
Parts:
- removed C6: 1u, Capacitors_SMD:C_0805_HandSoldering, symbol CP
- removed J4: Conn_01x03_Male, Pin_Headers:Pin_Header_Straight_1x03_Pitch2.54mm, symbol Conn_01x03_Male
- removed Q1: Q_NMOS_DGS, TO_SOT_Packages_SMD:SOT-23, symbol Q_NMOS_DGS
- removed R4: 100k, Resistors_SMD:R_0805_HandSoldering, symbol R
- removed R5: 5, Resistors_SMD:R_0805_HandSoldering, symbol R
- removed U3: accel, SMD_Packages:SOIC-8-N, symbol accel
- removed U5: EEPROM, lib:SO8, symbol EEPROM
- C1, C2, C3, C4, C5, C7: footprint Capacitors_SMD:C_0805_HandSoldering -> Capacitors_SMD:C_0603
- J2, J3: footprint Pin_Headers:Pin_Header_Straight_1x05_Pitch2.54mm -> lib:pin5
- R1, R2, R3: footprint Resistors_SMD:R_0805_HandSoldering -> Resistors_SMD:R_0603
Connections:
- wire segments 119 -> 82

Commit message: wip
Parts:
- removed C2: 0.1u, Capacitors_SMD:C_0603, symbol CP
- removed C4: 10u, Capacitors_SMD:C_0603, symbol CP
- removed U2: test, lib:QFN_28, symbol dsPIC33_qfn
- added U2: PIC16F15325, symbol PIC16F15325
Connections:
- net +3V3: now also U2.16 (VDD)
- net DEBUG: now also U2.4 (RC5)
- net MCLR: now also U2.3 (MCLR)
- net PGC: now also U2.11 (ICSPCLK)
- net PGD: now also U2.12 (ICSPDAT)
- net SCK: now also U2.9 (RC0)
- net SDI: now also U2.8 (RC1)
- net SDO: now also U2.7 (RC2)
- net U1RX: now also U2.6 (RC3)
- net U1TX: now also U2.5 (RC4)
- net VSS: now also U2.13 (VSS)
- net at U6.2 (CSB): now also U2.10 (RA2)
- net at R1.1, R2.2: now also U2.2 (RA4)
Other:
- moved on the sheet: C5, R3

Commit message: DEV1 basic
Parts:
- removed C1: 10u, Capacitors_SMD:C_0603, symbol CP
- removed J1: Conn_01x03_Male, Pin_Headers:Pin_Header_Straight_1x03_Pitch2.54mm, symbol Conn_01x03_Male
- removed R1: 200k, Resistors_SMD:R_0603, symbol R
- removed R2: 100k, Resistors_SMD:R_0603, symbol R
- removed U1: TLV760, TO_SOT_Packages_SMD:SOT-23, symbol TLV760
- added B1: 1632-holder, lib:1632-holder, symbol 1632-holder
- added U1: EEPROM, lib:SO8, symbol EEPROM
- U2: footprint (none) -> lib:UQFN_16
Connections:
- net +3V3: now also B1.2 (POS), U1.8 (VDD)
- net SCK: now also U1.6 (SCK)
- net SDI: now also U1.2 (SDO)
- net SDO: now also U1.5 (SDI)
- net VSS: now also B1.1 (GND), U1.4 (VSS)
- net EEPROM_CS: now reaches U2.2 (RA4)
- net EEPROM_CS: now also U1.1 (~CS)
- net EEPROM_HOLD: now reaches U2.1 (RA5)
- net EEPROM_HOLD: now also U1.3 (~WP), U1.7 (~HOLD)
Changed lines of the file:
@@
 EESchema Schematic File Version 2
+LIBS:altimeter-rescue
 LIBS:power
 LIBS:device
@@
 $EndDescr
 $Comp
-L VSS #PWR7
+L VSS #PWR01
 U 1 1 5AB5A9F9
 P 3550 850
-F 0 "#PWR7" H 3550 700 50  0001 C CNN
+F 0 "#PWR01" H 3550 700 50  0001 C CNN
 F 1 "VSS" H 3550 1000 50  0000 C CNN
 F 2 "" H 3550 850 50  0001 C CNN
@@
 $EndComp
 $Comp
-L +3.3V #PWR5
+L +3.3V #PWR02
 U 1 1 5AB5B67C
 P 2950 750
-F 0 "#PWR5" H 2950 600 50  0001 C CNN
+F 0 "#PWR02" H 2950 600 50  0001 C CNN
 F 1 "+3.3V" H 2950 890 50  0000 C CNN
 F 2 "" H 2950 750 50  0001 C CNN
@@
 $EndComp
 $Comp
-L +3.3V #PWR1
+L +3.3V #PWR03
 U 1 1 5ABE927B
 P 1300 2250
-F 0 "#PWR1" H 1300 2100 50  0001 C CNN
+F 0 "#PWR03" H 1300 2100 50  0001 C CNN
 F 1 "+3.3V" H 1300 2390 50  0000 C CNN
 F 2 "" H 1300 2250 50  0001 C CNN
@@
 U1RX
 $Comp
-L +3.3V #PWR9
+L +3.3V #PWR04
 U 1 1 5ABFEDB5
 P 5550 5200
-F 0 "#PWR9" H 5550 5050 50  0001 C CNN
+F 0 "#PWR04" H 5550 5050 50  0001 C CNN
 F 1 "+3.3V" H 5550 5340 50  0000 C CNN
 F 2 "" H 5550 5200 50  0001 C CNN
@@
 $EndComp
 $Comp
-L VSS #PWR10
+L VSS #PWR05
 U 1 1 5ABFEDDD
 P 5650 5350
-F 0 "#PWR10" H 5650 5200 50  0001 C CNN
+F 0 "#PWR05" H 5650 5200 50  0001 C CNN
 F 1 "VSS" H 5650 5500 50  0000 C CNN
 F 2 "" H 5650 5350 50  0001 C CNN
@@
 $EndComp
 $Comp
-L VSS #PWR8
+L VSS #PWR06
 U 1 1 5ABFF34C
 P 4150 5100
-F 0 "#PWR8" H 4150 4950 50  0001 C CNN
+F 0 "#PWR06" H 4150 4950 50  0001 C CNN
 F 1 "VSS" H 4150 5250 50  0000 C CNN
 F 2 "" H 4150 5100 50  0001 C CNN
@@
 PGD
 $Comp
-L +3.3V #PWR2
+L +3.3V #PWR07
 U 1 1 5AC12FB0
 P 2200 3900
-F 0 "#PWR2" H 2200 3750 50  0001 C CNN
+F 0 "#PWR07" H 2200 3750 50  0001 C CNN
 F 1 "+3.3V" H 2200 4040 50  0000 C CNN
 F 2 "" H 2200 3900 50  0001 C CNN
@@
 $EndComp
 $Comp
-L VSS #PWR3
+L VSS #PWR08
 U 1 1 5AC12FCE
 P 2450 4000
-F 0 "#PWR3" H 2450 3850 50  0001 C CNN
+F 0 "#PWR08" H 2450 3850 50  0001 C CNN
 F 1 "VSS" H 2450 4150 50  0000 C CNN
 F 2 "" H 2450 4000 50  0001 C CNN
@@
 PGD
 $Comp
-L +3.3V #PWR11
+L +3.3V #PWR09
 U 1 1 5AC190CB
 P 8150 900
-F 0 "#PWR11" H 8150 750 50  0001 C CNN
+F 0 "#PWR09" H 8150 750 50  0001 C CNN
 F 1 "+3.3V" H 8150 1040 50  0000 C CNN
 F 2 "" H 8150 900 50  0001 C CNN
@@
 $EndComp
 $Comp
-L VSS #PWR12
+L VSS #PWR010
 U 1 1 5AC190DC
 P 8400 2150
-F 0 "#PWR12" H 8400 2000 50  0001 C CNN
+F 0 "#PWR010" H 8400 2000 50  0001 C CNN
 F 1 "VSS" H 8400 2300 50  0000 C CNN
 F 2 "" H 8400 2150 50  0001 C CNN
@@
 $EndComp
 $Comp
-L TLV760 U1
-U 1 1 5AC196C8
-P 2350 5500
-F 0 "U1" H 2350 5500 39  0000 C CNN
-F 1 "TLV760" H 2350 5600 39  0000 C CNN
-F 2 "TO_SOT_Packages_SMD:SOT-23" H 2350 5500 39  0001 C CNN
-F 3 "" H 2350 5500 39  0001 C CNN
-	1    2350 5500
-	1    0    0    -1
-$EndComp
-$Comp
-L +3.3V #PWR6
+L +3.3V #PWR011
 U 1 1 5AC19B3B
 P 3150 5400
-F 0 "#PWR6" H 3150 5250 50  0001 C CNN
+F 0 "#PWR011" H 3150 5250 50  0001 C CNN
 F 1 "+3.3V" H 3150 5540 50  0000 C CNN
 F 2 "" H 3150 5400 50  0001 C CNN
@@
 $EndComp
 $Comp
-L VSS #PWR4
+L VSS #PWR012
 U 1 1 5AC19BAA
 P 2550 6050
-F 0 "#PWR4" H 2550 5900 50  0001 C CNN
+F 0 "#PWR012" H 2550 5900 50  0001 C CNN
 F 1 "VSS" H 2550 6200 50  0000 C CNN
 F 2 "" H 2550 6050 50  0001 C CNN
@@
 Text GLabel 1400 5500 0    39   Input ~ 0
 VIN
-$Comp
-L R R2
-U 1 1 5AC1A258
-P 2100 6050
-F 0 "R2" V 2180 6050 50  0000 C CNN
-F 1 "100k" V 2100 6050 50  0000 C CNN
-F 2 "Resistors_SMD:R_0603" V 2030 6050 50  0001 C CNN
-F 3 "" H 2100 6050 50  0001 C CNN
-	1    2100 6050
-	0    1    1    0
-$EndComp
-$Comp
-L R R1
-U 1 1 5AC1A296
-P 1750 6050
-F 0 "R1" V 1830 6050 50  0000 C CNN
-F 1 "200k" V 1750 6050 50  0000 C CNN
-F 2 "Resistors_SMD:R_0603" V 1680 6050 50  0001 C CNN
-F 3 "" H 1750 6050 50  0001 C CNN
-	1    1750 6050
-	0    1    1    0
-$EndComp
 $Comp
 L Conn_01x05_Male J3
@@
 	-1   0    0    -1
 $EndComp
-$Comp
-L Conn_01x03_Male J1
-U 1 1 5AC24686
-P 900 5900
-F 0 "J1" H 900 6100 50  0000 C CNN
-F 1 "Conn_01x03_Male" H 900 5700 50  0000 C CNN
-F 2 "Pin_Headers:Pin_Header_Straight_1x03_Pitch2.54mm" H 900 5900 50  0001 C CNN
-F 3 "" H 900 5900 50  0001 C CNN
-	1    900  5900
-	1    0    0    -1
-$EndComp
 Text GLabel 1250 5800 2    39   Input ~ 0
 DEBUG
 Text GLabel 2250 2550 0    39   Input ~ 0
 DEBUG
-$Comp
-L CP C1
-U 1 1 5AC2641C
-P 1500 6100
-F 0 "C1" H 1525 6200 50  0000 L CNN
-F 1 "10u" H 1525 6000 50  0000 L CNN
-F 2 "Capacitors_SMD:C_0603" H 1538 5950 50  0001 C CNN
-F 3 "" H 1500 6100 50  0001 C CNN
-	1    1500 6100
-	-1   0    0    -1
-$EndComp
 $Comp
 L CP C3
@@
 U 1 1 5B36ECB1
 P 3250 2250
-F 0 "U2" H 3250 2250 39  0000 C CNN
+F 0 "U2" H 3250 2350 39  0000 C CNN
 F 1 "PIC16F15325" H 3250 2250 39  0000 C CNN
-F 2 "" H 3250 2250 39  0001 C CNN
+F 2 "lib:UQFN_16" H 3250 2250 39  0001 C CNN
 F 3 "" H 3250 2250 39  0001 C CNN
 	1    3250 2250
@@
 	3150 5400 3150 5750
 Wire Wire Line
-	2350 6350 2350 5950
-Wire Wire Line
-	2250 6050 2550 6050
-Connection ~ 2350 6050
-Wire Wire Line
-	1950 6050 1900 6050
-Wire Wire Line
-	1600 5500 1600 6050
-Connection ~ 1600 5500
-Wire Wire Line
-	1950 2100 1950 6050
-Wire Wire Line
 	5600 5950 4950 5950
 Wire Wire Line
@@
 	5400 5750 5600 5750
 Wire Wire Line
-	1100 5900 1600 5900
-Connection ~ 1600 5900
-Wire Wire Line
-	1100 6000 1300 6000
-Wire Wire Line
-	1300 6000 1300 6350
-Wire Wire Line
-	1300 6350 3150 6350
-Wire Wire Line
 	1250 5800 1100 5800
 Wire Wire Line
 	2450 2550 2250 2550
-Wire Wire Line
-	1500 5950 1500 5900
-Connection ~ 1500 5900
-Wire Wire Line
-	1500 6250 1500 6350
-Connection ~ 1500 6350
 Connection ~ 3150 5500
 Wire Wire Line
 	3150 6350 3150 6050
-Connection ~ 2350 6350
 Wire Wire Line
 	9300 1000 9300 1250
@@
 Connection ~ 3550 850
 Wire Wire Line
-	2950 5500 3150 5500
-Wire Wire Line
-	1400 5500 1750 5500
+	1400 5500 3150 5500
 Wire Wire Line
 	2950 3200 2950 3050
@@
 Wire Wire Line
 	1750 2300 1750 2400
-Wire Wire Line
-	1950 2100 2450 2100
+$Comp
+L 1632-holder B1
+U 1 1 5B3ED464
+P 5400 3600
+F 0 "B1" H 5400 3600 60  0000 C CNN
+F 1 "1632-holder" H 5400 3600 60  0000 C CNN
+F 2 "lib:1632-holder" H 5400 3600 60  0001 C CNN
+F 3 "" H 5400 3600 60  0001 C CNN
+	1    5400 3600
+	1    0    0    -1
+$EndComp
+$Comp
+L +3.3V #PWR013
+U 1 1 5B3ED514
+P 6200 3200
+F 0 "#PWR013" H 6200 3050 50  0001 C CNN
+F 1 "+3.3V" H 6200 3340 50  0000 C CNN
+F 2 "" H 6200 3200 50  0001 C CNN
+F 3 "" H 6200 3200 50  0001 C CNN
+	1    6200 3200
+	1    0    0    -1
+$EndComp
+$Comp
+L VSS #PWR014
+U 1 1 5B3ED538
+P 4550 3200
+F 0 "#PWR014" H 4550 3050 50  0001 C CNN
+F 1 "VSS" H 4550 3350 50  0000 C CNN
+F 2 "" H 4550 3200 50  0001 C CNN
+F 3 "" H 4550 3200 50  0001 C CNN
+	1    4550 3200
+	1    0    0    -1
+$EndComp
+Wire Wire Line
+	6200 3200 6200 3300
+Wire Wire Line
+	6200 3300 6000 3300
+Wire Wire Line
+	4550 3200 4550 3300
+Wire Wire Line
+	4550 3300 4750 3300
+Wire Wire Line
+	2550 6050 2550 6350
+Connection ~ 2550 6350
+Wire Wire Line
+	2550 6350 3150 6350
+$Comp
+L EEPROM U1
+U 1 1 5BB6D30E
+P 8200 3000
+F 0 "U1" H 7900 3250 50  0000 L CNN
+F 1 "EEPROM" H 8250 3250 50  0000 L CNN
+F 2 "lib:SO8" H 7850 2950 50  0001 C CNN
+F 3 "" H 7850 2950 50  0001 C CNN
+	1    8200 3000
+	1    0    0    -1
+$EndComp
+Text GLabel 7450 3100 0    39   Input ~ 0
+EEPROM_CS
+Text GLabel 7450 3000 0    39   Input ~ 0
+EEPROM_HOLD
+Text GLabel 8700 2900 2    39   Input ~ 0
+SCK
+Text GLabel 8700 3100 2    39   Output ~ 0
+SDI
+Text GLabel 8700 3000 2    39   Input ~ 0
+SDO
+Wire Wire Line
+	8600 2900 8700 2900
+Wire Wire Line
+	8600 3000 8700 3000
+Wire Wire Line
+	8600 3100 8700 3100
+Wire Wire Line
+	7450 3000 7800 3000
+Wire Wire Line
+	7450 3100 7800 3100
+$Comp
+L +3.3V #PWR015
+U 1 1 5BB6D739
+P 8200 2550
+F 0 "#PWR015" H 8200 2400 50  0001 C CNN
+F 1 "+3.3V" H 8200 2690 50  0000 C CNN
+F 2 "" H 8200 2550 50  0001 C CNN
+F 3 "" H 8200 2550 50  0001 C CNN
+	1    8200 2550
+	1    0    0    -1
+$EndComp
+$Comp
+L VSS #PWR016
+U 1 1 5BB6D793
+P 8400 3450
+F 0 "#PWR016" H 8400 3300 50  0001 C CNN
+F 1 "VSS" H 8400 3600 50  0000 C CNN
+F 2 "" H 8400 3450 50  0001 C CNN
+F 3 "" H 8400 3450 50  0001 C CNN
+	1    8400 3450
+	1    0    0    -1
+$EndComp
+Wire Wire Line
+	8200 3300 8200 3450
+Wire Wire Line
+	8200 3450 8400 3450
+Text GLabel 7450 2900 0    39   Input ~ 0
+EEPROM_WP
+Wire Wire Line
+	7800 2900 7450 2900
+Wire Wire Line
+	7650 2900 7650 3000
+Connection ~ 7650 3000
+Connection ~ 7650 2900
+Text GLabel 2300 2100 0    39   Input ~ 0
+EEPROM_CS
+Text GLabel 2300 1950 0    39   Input ~ 0
+EEPROM_HOLD
+Wire Wire Line
+	2300 1950 2450 1950
+Wire Wire Line
+	2300 2100 2450 2100
+Wire Wire Line
+	8200 2550 8200 2700
 $EndSCHEMATC
